File: ProtoGuitarPedalBoard.kicad_pcb (KiCad board)
At the start: 2 copper layers, 195 x 100 mm, 24 parts, among them J1 DC_INPUT

Commit message: Make PCB
Parts:
- J2: renamed from J_Signal_Effect_IN1; value Conn_01x02 -> FX_IN
- J3: renamed from J_Signal_Effect_OUT1; value Conn_01x02 -> FX_OUT
- moved J_POT4 373.8 mm to (314.0, 183.5), turned to 180 degrees
- moved J_POT3 366.3 mm to (314.0, 148.6), turned to 180 degrees
- moved J_POT2 223.7 mm to (136.0, 178.5)
- moved J_POT1 208.2 mm to (136.0, 143.5)
- moved H1 18.5 mm to (117.0, 105.5)
- moved H3 17.8 mm to (117.0, 193.5)
- moved POT2 15.3 mm to (128.7, 178.5)
- moved POT1 15.1 mm to (128.7, 143.5)
- moved H2 13.9 mm to (333.0, 105.5)
- moved H4 12.9 mm to (333.0, 193.5)
- moved R2 12.3 mm to (232.5, 112.4), turned to -90 degrees
- moved POT4 10.6 mm to (321.3, 183.5)
- moved SW_3PDT_ToggleBtn1 10.5 mm to (257.2, 117.0)
- moved POT3 10.5 mm to (321.3, 148.6)
- moved D1_Green_LED1 7.02 mm to (207.0, 123.5)
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- renumbered J_R_POT_1 to J_POT1, J_R_POT_2 to J_POT2, J_R_POT_3 to J_POT3, J_R_POT_4 to J_POT4, RV1 to POT1, RV2 to POT2, RV3 to POT3, RV4 to POT4
Other:
- board size 195 x 100 mm -> 225 x 97 mm
- board text added: "<- ->"
- board text added: "Bread Board 164 x 54 [mm]"
- board text added: "GND"
- board text added: "Guitar Effect"
- board text added: "Jack Input"
- board text added: "Jack Output"
- board text added: "ON/OFF"
- board text added: "ON/OFF (DC Power)"
- board text added: "ON/OFF (Guitar Effect)"
- board text added: "Out1"
- board text added: "Out2"
- board text added: "Out3"
- board text added: "Out4"
- board text added: "VCC"

Commit message: Update
Parts:
- moved J_POT1 5.09 mm to (136.0, 148.6), turned to 180 degrees
- moved J_POT2 5.06 mm to (135.9, 183.5), turned to 180 degrees
Connections:
- J2 pad 1: /Signal_Effect_IN -> GND
- J2 pad 2: GND -> /Signal_Effect_IN
- J3 pad 1: /Signal_Effect_OUT -> GND
- J3 pad 2: GND -> /Signal_Effect_OUT
- J_POT1 pad 1: /Vcc1 -> /GND_1
- J_POT1 pad 3: /GND_1 -> /Vcc1
- J_POT2 pad 1: /Vcc2 -> /GND_2
- J_POT2 pad 3: /GND_2 -> /Vcc2
- J_POT3 pad 1: /Vcc3 -> /GND_3
- J_POT3 pad 3: /GND_3 -> /Vcc3
- J_POT4 pad 1: /Vcc4 -> /GND_4
- J_POT4 pad 3: /GND_4 -> /Vcc4
Changed lines of the file:
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@@
 	(footprint "Connector_PinSocket_2.54mm:PinSocket_1x03_P2.54mm_Vertical"
 		(layer "F.Cu")
-		(at 314 183.54 180)
+		(at 314 183.515 180)
 		(descr "Through hole straight socket strip, 1x03, 2.54mm pitch, single row (from Kicad 4.0.7), script generated")
 		(tags "Through hole socket strip THT 1x03 2.54mm single row")
@@
 			(layers "*.Cu" "*.Mask")
 			(remove_unused_layers no)
-			(net "/Vcc4")
+			(net "/GND_4")
 			(pinfunction "Pin_1_1")
 			(pintype "passive")
@@
 			(layers "*.Cu" "*.Mask")
 			(remove_unused_layers no)
-			(net "/GND_4")
+			(net "/Vcc4")
 			(pinfunction "Pin_3_3")
 			(pintype "passive")
@@
 	(footprint "Connector_PinSocket_2.54mm:PinSocket_1x03_P2.54mm_Vertical"
 		(layer "F.Cu")
-		(at 314 148.58 180)
+		(at 314 148.59 180)
 		(descr "Through hole straight socket strip, 1x03, 2.54mm pitch, single row (from Kicad 4.0.7), script generated")
 		(tags "Through hole socket strip THT 1x03 2.54mm single row")
@@
 			(layers "*.Cu" "*.Mask")
 			(remove_unused_layers no)
-			(net "/Vcc3")
+			(net "/GND_3")
 			(pinfunction "Pin_1_1")
 			(pintype "passive")
@@
 			(layers "*.Cu" "*.Mask")
 			(remove_unused_layers no)
-			(net "/GND_3")
+			(net "/Vcc3")
 			(pinfunction "Pin_3_3")
 			(pintype "passive")
@@
 	(footprint "Connector_PinSocket_2.54mm:PinSocket_1x03_P2.54mm_Vertical"
 		(layer "F.Cu")
-		(at 136 143.5)
+		(at 136 148.59 180)
 		(descr "Through hole straight socket strip, 1x03, 2.54mm pitch, single row (from Kicad 4.0.7), script generated")
 		(tags "Through hole socket strip THT 1x03 2.54mm single row")
 		(property "Reference" "J_POT1"
-			(at 0 -2.77 0)
+			(at 0 7.86 0)
 			(layer "F.SilkS")
 			(effects
@@
 		)
 		(property "Value" "Conn_01x03"
-			(at 0 7.85 0)
+			(at 0 -2.76 0)
 			(layer "F.Fab")
 			(effects
@@
 		(duplicate_pad_numbers_are_jumpers no)
 		(fp_line
-			(start -1.33 1.27)
-			(end -1.33 6.41)
+			(start 1.33 1.27)
+			(end 1.33 6.41)
 			(stroke
 				(width 0.12)
@@
 		)
 		(fp_line
-			(start -1.33 1.27)
-			(end 1.33 1.27)
+			(start 1.33 -1.33)
+			(end 1.33 0)
 			(stroke
 				(width 0.12)
@@
 		)
 		(fp_line
-			(start -1.33 6.41)
-			(end 1.33 6.41)
+			(start 0 -1.33)
+			(end 1.33 -1.33)
 			(stroke
 				(width 0.12)
@@
 		)
 		(fp_line
-			(start 0 -1.33)
-			(end 1.33 -1.33)
+			(start -1.33 6.41)
+			(end 1.33 6.41)
 			(stroke
 				(width 0.12)
@@
 		)
 		(fp_line
-			(start 1.33 -1.33)
-			(end 1.33 0)
+			(start -1.33 1.27)
+			(end 1.33 1.27)
 			(stroke
 				(width 0.12)
@@
 		)
 		(fp_line
-			(start 1.33 1.27)
-			(end 1.33 6.41)
+			(start -1.33 1.27)
+			(end -1.33 6.41)
 			(stroke
 				(width 0.12)
@@
 		)
 		(fp_line
-			(start -1.77 -1.77)
-			(end 1.77 -1.77)
+			(start 1.77 6.85)
+			(end -1.77 6.85)
 			(stroke
 				(width 0.05)
@@
 		)
 		(fp_line
-			(start -1.77 6.85)
-			(end -1.77 -1.77)
+			(start 1.77 -1.77)
+			(end 1.77 6.85)
 			(stroke
 				(width 0.05)
@@
 		)
 		(fp_line
-			(start 1.77 -1.77)
-			(end 1.77 6.85)
+			(start -1.77 6.85)
+			(end -1.77 -1.77)
 			(stroke
 				(width 0.05)
@@
 		)
 		(fp_line
-			(start 1.77 6.85)
-			(end -1.77 6.85)
+			(start -1.77 -1.77)
+			(end 1.77 -1.77)
 			(stroke
 				(width 0.05)
@@
 		)
 		(fp_line
-			(start -1.27 -1.27)
-			(end 0.635 -1.27)
+			(start 1.27 6.35)
+			(end -1.27 6.35)
 			(stroke
 				(width 0.1)
@@
 		)
 		(fp_line
-			(start -1.27 6.35)
-			(end -1.27 -1.27)
+			(start 1.27 -0.635)
+			(end 1.27 6.35)
 			(stroke
 				(width 0.1)
@@
 		)
 		(fp_line
-			(start 1.27 -0.635)
-			(end 1.27 6.35)
+			(start -1.27 6.35)
+			(end -1.27 -1.27)
 			(stroke
 				(width 0.1)
@@
 		)
 		(fp_line
-			(start 1.27 6.35)
-			(end -1.27 6.35)
+			(start -1.27 -1.27)
+			(end 0.635 -1.27)
 			(stroke
 				(width 0.1)
@@
 		)
 		(pad "1" thru_hole rect
-			(at 0 0)
+			(at 0 0 180)
 			(size 1.7 1.7)
 			(drill 1)
 			(layers "*.Cu" "*.Mask")
 			(remove_unused_layers no)
-			(net "/Vcc1")
+			(net "/GND_1")
 			(pinfunction "Pin_1_1")
 			(pintype "passive")
 		)
 		(pad "2" thru_hole circle
-			(at 0 2.54)
+			(at 0 2.54 180)
 			(size 1.7 1.7)
 			(drill 1)
@@
 		)
 		(pad "3" thru_hole circle
-			(at 0 5.08)
+			(at 0 5.08 180)
 			(size 1.7 1.7)
 			(drill 1)
 			(layers "*.Cu" "*.Mask")
 			(remove_unused_layers no)
-			(net "/GND_1")
+			(net "/Vcc1")
 			(pinfunction "Pin_3_3")
 			(pintype "passive")
@@
 			(layers "*.Cu" "*.Mask")
 			(remove_unused_layers no)
-			(net "/Signal_Effect_IN")
+			(net "GND")
 			(pinfunction "Pin_1_1")
 			(pintype "passive")
@@
 			(layers "*.Cu" "*.Mask")
 			(remove_unused_layers no)
-			(net "GND")
+			(net "/Signal_Effect_IN")
 			(pinfunction "Pin_2_2")
 			(pintype "passive")
@@
 			(layers "*.Cu" "*.Mask")
 			(remove_unused_layers no)
-			(net "/Signal_Effect_OUT")
+			(net "GND")
 			(pinfunction "Pin_1_1")
 			(pintype "passive")
@@
 			(layers "*.Cu" "*.Mask")
 			(remove_unused_layers no)
-			(net "GND")
+			(net "/Signal_Effect_OUT")
 			(pinfunction "Pin_2_2")
 			(pintype "passive")
@@
 	(footprint "Connector_PinSocket_2.54mm:PinSocket_1x03_P2.54mm_Vertical"
 		(layer "F.Cu")
-		(at 136 178.46)
+		(at 135.89 183.515 180)
 		(descr "Through hole straight socket strip, 1x03, 2.54mm pitch, single row (from Kicad 4.0.7), script generated")
 		(tags "Through hole socket strip THT 1x03 2.54mm single row")
 		(property "Reference" "J_POT2"
-			(at 0 -2.77 0)
+			(at 0 7.825 0)
 			(layer "F.SilkS")
 			(effects
@@
 		)
 		(property "Value" "Conn_01x03"
-			(at 0 7.85 0)
+			(at 0 -2.795 0)
 			(layer "F.Fab")
 			(effects
@@
 		(duplicate_pad_numbers_are_jumpers no)
 		(fp_line
-			(start -1.33 1.27)
-			(end -1.33 6.41)
+			(start 1.33 1.27)
+			(end 1.33 6.41)
 			(stroke
 				(width 0.12)
@@
 		)
 		(fp_line
-			(start -1.33 1.27)
-			(end 1.33 1.27)
+			(start 1.33 -1.33)
+			(end 1.33 0)
 			(stroke
 				(width 0.12)
@@
 		)
 		(fp_line
-			(start -1.33 6.41)
-			(end 1.33 6.41)
+			(start 0 -1.33)
+			(end 1.33 -1.33)
 			(stroke
 				(width 0.12)
@@
 		)
 		(fp_line
-			(start 0 -1.33)
-			(end 1.33 -1.33)
+			(start -1.33 6.41)
+			(end 1.33 6.41)
 			(stroke
 				(width 0.12)
@@
 		)
 		(fp_line
-			(start 1.33 -1.33)
-			(end 1.33 0)
+			(start -1.33 1.27)
+			(end 1.33 1.27)
 			(stroke
 				(width 0.12)
@@
 		)
 		(fp_line
-			(start 1.33 1.27)
-			(end 1.33 6.41)
+			(start -1.33 1.27)
+			(end -1.33 6.41)
 			(stroke
 				(width 0.12)
@@
 		)
 		(fp_line
-			(start -1.77 -1.77)
-			(end 1.77 -1.77)
+			(start 1.77 6.85)
+			(end -1.77 6.85)
 			(stroke
 				(width 0.05)
@@
 		)
 		(fp_line
-			(start -1.77 6.85)
-			(end -1.77 -1.77)
+			(start 1.77 -1.77)
+			(end 1.77 6.85)
 			(stroke
 				(width 0.05)
@@
 		)
 		(fp_line
-			(start 1.77 -1.77)
-			(end 1.77 6.85)
+			(start -1.77 6.85)
+			(end -1.77 -1.77)
 			(stroke
 				(width 0.05)
@@
 		)
 		(fp_line
-			(start 1.77 6.85)
-			(end -1.77 6.85)
+			(start -1.77 -1.77)
+			(end 1.77 -1.77)
 			(stroke
 				(width 0.05)
@@
 		)
 		(fp_line
-			(start -1.27 -1.27)
-			(end 0.635 -1.27)
+			(start 1.27 6.35)
+			(end -1.27 6.35)
 			(stroke
 				(width 0.1)
@@
 		)
 		(fp_line
-			(start -1.27 6.35)
-			(end -1.27 -1.27)
+			(start 1.27 -0.635)
+			(end 1.27 6.35)
 			(stroke
 				(width 0.1)
@@
 		)
 		(fp_line
-			(start 1.27 -0.635)
-			(end 1.27 6.35)
+			(start -1.27 6.35)
+			(end -1.27 -1.27)
 			(stroke
 				(width 0.1)
@@
 		)
 		(fp_line
-			(start 1.27 6.35)
-			(end -1.27 6.35)
+			(start -1.27 -1.27)
+			(end 0.635 -1.27)
 			(stroke
 				(width 0.1)
@@
 		)
 		(pad "1" thru_hole rect
-			(at 0 0)
+			(at 0 0 180)
 			(size 1.7 1.7)
 			(drill 1)
 			(layers "*.Cu" "*.Mask")
 			(remove_unused_layers no)
-			(net "/Vcc2")
+			(net "/GND_2")
 			(pinfunction "Pin_1_1")
 			(pintype "passive")
 		)
 		(pad "2" thru_hole circle
-			(at 0 2.54)
+			(at 0 2.54 180)
 			(size 1.7 1.7)
 			(drill 1)
@@
 		)
 		(pad "3" thru_hole circle
-			(at 0 5.08)
+			(at 0 5.08 180)
 			(size 1.7 1.7)
 			(drill 1)
 			(layers "*.Cu" "*.Mask")
 			(remove_unused_layers no)
-			(net "/GND_2")
+			(net "/Vcc2")
 			(pinfunction "Pin_3_3")
 			(pintype "passive")
@@
 		)
 	)
-	(gr_text "VCC"
+	(gr_text "GND"
 		(at 139 161.5 0)
 		(layer "F.SilkS")
@@
 		)
 	)
-	(gr_text "GND"
+	(gr_text "VCC"
 		(at 139 164.5 0)
 		(layer "F.SilkS")
@@
 		)
 	)
-	(gr_text "GND"
+	(gr_text "VCC"
 		(at 311 143.5 0)
 		(layer "F.SilkS")
@@
 		)
 	)
-	(gr_text "VCC"
+	(gr_text "GND"
 		(at 311 148.5 0)
 		(layer "F.SilkS")
@@
 		)
 	)
-	(gr_text "VCC"
+	(gr_text "GND"
 		(at 311 161.5 0)
 		(layer "F.SilkS")
@@
 		)
 	)
-	(gr_text "GND"
+	(gr_text "VCC"
 		(at 311 164.5 0)
 		(layer "F.SilkS")
@@
 		)
 	)
-	(gr_text "GND"
+	(gr_text "VCC"
 		(at 311 178.5 0)
 		(layer "F.SilkS")
@@
 		)
 	)
-	(gr_text "VCC"
+	(gr_text "GND"
 		(at 311 183.5 0)
 		(layer "F.SilkS")

Commit message: End
Connections:
- net /GND_1 renamed /POT1_3
- net /GND_2 renamed /POT2_3
- net /Out1 renamed /POT1_2
- net /Out2 renamed /POT2_2
- net /Out3 renamed /POT3_2
- net /Out4 renamed /POT4_2
- net /Vcc1 renamed /POT1_1
- net /Vcc2 renamed /POT2_1
- J_POT3 pad 1: /GND_3 -> /POT3_3
- J_POT3 pad 3: /Vcc3 -> /POT3_1
- J_POT4 pad 1: /GND_4 -> /POT4_3
- J_POT4 pad 3: /Vcc4 -> /POT4_1
- POT3 pad 1: /Vcc3 -> /POT3_3
- POT3 pad 3: /GND_3 -> /POT3_1
- POT4 pad 1: /Vcc4 -> /POT4_3
- POT4 pad 3: /GND_4 -> /POT4_1
Routing:
- net /Signal_Effect_IN: track 0.00 -> 137.5 mm
- net /Signal_IN: track 0.00 -> 116.6 mm
- net /DC_OUT: track 0.00 -> 96.9 mm
- net /Signal_Effect_OUT: track 0.00 -> 75.2 mm
- net +9V: track 0.00 -> 48.8 mm
- net /OUT_2_LED_PWR: track 0.00 -> 31.3 mm, vias 0 -> 1
- net /Signal_OUT: track 0.00 -> 31.0 mm
- net /LED_RED: track 0.00 -> 20.2 mm
- net Net-(D1_Green_LED1-A): track 0.00 -> 14.4 mm
- net /Bypass: track 0.00 -> 12.7 mm
- net Net-(D2_Red_LED1-A): track 0.00 -> 10.1 mm
- net /POT3_1: track 0.00 -> 7.34 mm
- net /POT1_1: track 0.00 -> 7.34 mm
- net /POT3_2: track 0.00 -> 7.33 mm
- net /POT1_2: track 0.00 -> 7.33 mm
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- added copper zone on B.Cu, net GND
- added copper zone on F.Cu, net GND
Other:
- board text added: "POT1 1"
- board text added: "POT1 2"
- board text added: "POT1 3"
- board text added: "POT2 1"
- board text added: "POT2 2"
- board text added: "POT2 3"
- board text added: "POT3 1"
- board text added: "POT3 2"
- board text added: "POT3 3"
- board text added: "POT4 1"
- board text added: "POT4 2"
- board text added: "POT4 3"
- board text added: "Signal In"
- board text added: "Signal Out"
- board text removed: "Out1"
- board text removed: "Out2"
- board text removed: "Out3"
- board text removed: "Out4"

Commit message: Update routing pcb
Routing:
- net /Signal_Effect_OUT: track 75.2 -> 83.2 mm, vias 0 -> 1
- net /Signal_OUT: track 31.0 -> 24.0 mm
- net /OUT_2_LED_PWR: track 31.3 -> 28.4 mm
- net /Signal_IN: track 116.6 -> 119.4 mm
- net /Bypass: track 12.7 -> 13.5 mm
Changed lines of the file:
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@@
 	)
 	(segment
-		(start 196.215 113.625)
-		(end 196.215 110.49)
+		(start 186.34 123.5)
+		(end 196.85 112.99)
 		(width 0.7)
 		(layer "F.Cu")
@@
 	)
 	(segment
-		(start 186.34 123.5)
-		(end 196.215 113.625)
+		(start 196.85 112.99)
+		(end 196.85 112.97)
 		(width 0.7)
 		(layer "F.Cu")
@@
 	)
 	(via
-		(at 196.215 110.49)
+		(at 196.85 112.97)
 		(size 0.6)
 		(drill 0.3)
@@
 	)
 	(segment
-		(start 196.215 110.49)
-		(end 201.955 104.75)
+		(start 200.53 112.97)
+		(end 207.5 106)
 		(width 0.7)
 		(layer "B.Cu")
@@
 	)
 	(segment
-		(start 206.25 104.75)
-		(end 207.5 106)
-		(width 0.7)
-		(layer "B.Cu")
-		(net "/OUT_2_LED_PWR")
-	)
-	(segment
-		(start 201.955 104.75)
-		(end 206.25 104.75)
+		(start 196.85 112.97)
+		(end 200.53 112.97)
 		(width 0.7)
 		(layer "B.Cu")
@@
 	)
 	(segment
-		(start 282.945 109.855)
-		(end 261.62 109.855)
-		(width 0.3)
-		(layer "B.Cu")
-		(net "/Signal_OUT")
-	)
-	(segment
-		(start 283.3 109.5)
-		(end 282.945 109.855)
-		(width 0.3)
-		(layer "B.Cu")
-		(net "/Signal_OUT")
-	)
-	(segment
-		(start 261.62 109.855)
-		(end 259.715 111.76)
-		(width 0.3)
-		(layer "B.Cu")
-		(net "/Signal_OUT")
-	)
-	(segment
 		(start 262.440014 117.025014)
 		(end 262.525014 117.025014)
@@
 	)
 	(segment
-		(start 259.715 114.3)
-		(end 262.440014 117.025014)
+		(start 267.094986 117.025014)
+		(end 274.62 109.5)
 		(width 0.3)
 		(layer "B.Cu")
@@
 	)
 	(segment
-		(start 259.715 111.76)
-		(end 259.715 114.3)
+		(start 262.525014 117.025014)
+		(end 267.094986 117.025014)
+		(width 0.3)
+		(layer "B.Cu")
+		(net "/Signal_OUT")
+	)
+	(segment
+		(start 283.3 109.5)
+		(end 274.62 109.5)
 		(width 0.3)
 		(layer "B.Cu")
@@
 	)
 	(segment
-		(start 161.84 138.43)
-		(end 225.720028 138.43)
+		(start 136 164.27)
+		(end 200.5 164.27)
 		(width 0.3)
 		(layer "B.Cu")
@@
 	)
 	(segment
-		(start 136 164.27)
-		(end 161.84 138.43)
+		(start 200.5 164.27)
+		(end 251.925014 112.844986)
 		(width 0.3)
 		(layer "B.Cu")
@@
 	)
 	(segment
-		(start 225.720028 138.43)
+		(start 251.925014 112.844986)
 		(end 251.925014 112.225014)
 		(width 0.3)
@@
 	)
 	(segment
-		(start 156.495 103.505)
-		(end 150.5 109.5)
+		(start 150.5 109.5)
+		(end 156.98 103.02)
 		(width 0.3)
 		(layer "B.Cu")
@@
 	)
 	(segment
-		(start 252.095 109.22)
-		(end 219.075 109.22)
+		(start 254.56 107.11)
+		(end 254.56 114.390028)
 		(width 0.3)
 		(layer "B.Cu")
@@
 	)
 	(segment
-		(start 251.925014 117.025014)
-		(end 254.875014 114.075014)
+		(start 156.98 103.02)
+		(end 250.47 103.02)
 		(width 0.3)
 		(layer "B.Cu")
@@
 	)
 	(segment
-		(start 213.36 103.505)
-		(end 156.495 103.505)
+		(start 254.56 114.390028)
+		(end 251.925014 117.025014)
 		(width 0.3)
 		(layer "B.Cu")
@@
 	)
 	(segment
-		(start 219.075 109.22)
-		(end 213.36 103.505)
+		(start 250.47 103.02)
+		(end 254.56 107.11)
 		(width 0.3)
 		(layer "B.Cu")
@@
 	)
 	(segment
-		(start 254.875014 114.075014)
-		(end 254.875014 112.000014)
-		(width 0.3)
-		(layer "B.Cu")
-		(net "/Signal_IN")
-	)
-	(segment
-		(start 254.875014 112.000014)
-		(end 252.095 109.22)
-		(width 0.3)
-		(layer "B.Cu")
-		(net "/Signal_IN")
-	)
-	(segment
-		(start 253.350014 123.250014)
-		(end 261.100014 123.250014)
+		(start 259.19 124.16)
+		(end 261.524986 121.825014)
 		(width 0.2)
 		(layer "B.Cu")
@@
 	)
 	(segment
-		(start 261.100014 123.250014)
+		(start 254.26 124.16)
+		(end 259.19 124.16)
+		(width 0.2)
+		(layer "B.Cu")
+		(net "/Bypass")
+	)
+	(segment
+		(start 261.524986 121.825014)
 		(end 262.525014 121.825014)
 		(width 0.2)
@@
 	(segment
 		(start 251.925014 121.825014)
-		(end 253.350014 123.250014)
+		(end 254.26 124.16)
 		(width 0.2)
 		(layer "B.Cu")
@@
 	)
 	(segment
+		(start 270.87 119.93)
+		(end 263.165014 112.225014)
+		(width 0.3)
+		(layer "F.Cu")
+		(net "/Signal_Effect_OUT")
+	)
+	(segment
+		(start 263.165014 112.225014)
+		(end 262.525014 112.225014)
+		(width 0.3)
+		(layer "F.Cu")
+		(net "/Signal_Effect_OUT")
+	)
+	(segment
 		(start 262.525014 112.225014)
 		(end 264.125014 112.225014)
@@
 		(net "/Signal_Effect_OUT")
 	)
+	(via
+		(at 270.87 119.93)
+		(size 0.6)
+		(drill 0.3)
+		(layers "F.Cu" "B.Cu")
+		(net "/Signal_Effect_OUT")
+	)
+	(segment
+		(start 270.87 129.94)
+		(end 305.2 164.27)
+		(width 0.3)
+		(layer "B.Cu")
+		(net "/Signal_Effect_OUT")
+	)
+	(segment
+		(start 270.87 119.93)
+		(end 270.87 129.94)
+		(width 0.3)
+		(layer "B.Cu")
+		(net "/Signal_Effect_OUT")
+	)
+	(segment
+		(start 305.2 164.27)
+		(end 314 164.27)
+		(width 0.3)
+		(layer "B.Cu")
+		(net "/Signal_Effect_OUT")
+	)
 	(segment
 		(start 262.525014 112.225014)
@@
 	)
 	(segment
-		(start 262.525014 112.795014)
-		(end 314 164.27)
-		(width 0.2)
+		(start 262.525014 112.225014)
+		(end 262.525014 112.385014)
+		(width 0.2)
+		(layer "B.Cu")
+		(net "/Signal_Effect_OUT")
+	)
+	(segment
+		(start 264.325014 112.225014)
+		(end 262.525014 112.225014)
+		(width 0.3)
 		(layer "B.Cu")
 		(net "/Signal_Effect_OUT")
@@
 		(polygon
 			(pts
-				(xy 107.95 95.25) (xy 342.9 95.25) (xy 342.9 203.2) (xy 107.95 203.2)
+				(xy 110 90.02) (xy 347.76 90.14) (xy 350.23 202.81) (xy 107.94 205.88) (xy 110.11 89.98)
 			)
 		)
