File: ProtoGuitarPedalBoard.kicad_pcb (KiCad board)
At the start: 2 copper layers, 225 x 97 mm, 24 parts, among them J1 DC_INPUT, J2 FX_IN, J3 FX_OUT

Commit message: Reset PCB routing
Routing:
- net /Signal_Effect_IN: track 137.8 -> 0.62 mm
- net /Signal_IN: track 119.4 -> 0.00 mm
- net /DC_OUT: track 96.9 -> 0.00 mm
- net /Signal_Effect_OUT: track 83.2 -> 4.97 mm, vias 1 -> 0
- net +9V: track 48.8 -> 1.30 mm
- net /OUT_2_LED_PWR: track 28.4 -> 0.00 mm, vias 1 -> 0
- net /Signal_OUT: track 24.0 -> 0.08 mm
- net /LED_RED: track 20.2 -> 3.26 mm
- net Net-(D1_Green_LED1-A): track 14.4 -> 1.90 mm
- net /Bypass: track 13.5 -> 1.95 mm
- net Net-(D2_Red_LED1-A): track 10.1 -> 0.00 mm
- net /POT4_3: track 7.32 -> 0.00 mm
- net /POT4_2: track 7.32 -> 0.00 mm
- net /POT4_1: track 7.32 -> 0.00 mm
- net /POT3_3: track 7.33 -> 0.01 mm
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- removed copper zone on B.Cu, net GND
- removed copper zone on F.Cu, net GND

Commit message: Final PCB layout: complete routing, copper pour, and zero DRC errors
Parts:
- moved H1 0.55 mm to (116.8, 105.0)
- moved H4 0.55 mm to (333.2, 194.0)
- moved H3 0.53 mm to (116.8, 194.0)
- moved H2 0.51 mm to (333.2, 105.0)
Routing:
- net /Signal_Effect_IN: track 0.62 -> 137.5 mm
- net /Signal_IN: track 0.00 -> 120.3 mm
- net /DC_OUT: track 0.00 -> 83.7 mm
- net /Signal_Effect_OUT: track 4.97 -> 73.4 mm
- net +9V: track 1.30 -> 55.7 mm
- net /Signal_OUT: track 0.08 -> 31.5 mm
- net /OUT_2_LED_PWR: track 0.00 -> 28.4 mm
- net /LED_RED: track 3.26 -> 20.3 mm
- net Net-(D1_Green_LED1-A): track 1.90 -> 14.8 mm
- net /Bypass: track 1.95 -> 12.7 mm
- net Net-(D2_Red_LED1-A): track 0.00 -> 10.1 mm
- net /POT4_3: track 0.00 -> 7.32 mm
- net /POT4_2: track 0.00 -> 7.32 mm
- net /POT4_1: track 0.00 -> 7.32 mm
- net /POT3_3: track 0.01 -> 7.33 mm
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- added copper zone on B.Cu, net GND
- added copper zone on F.Cu, net GND
Other:
- board text added: "DC_OUT"
- board text added: "Green LED"
- board text added: "Red LED"

Commit message: Add Breadboard 3d_model, symbol and footprint, add breadboard on the pcb
Parts:
- added U1: Bread Board, MyFootPrints:Breadboard, F.Cu at (225.0, 166.0)
Changed lines of the file:
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@@
 		(capping no)
 		(filling no)
-		(zone_defaults)
 		(pcbplotparams
 			(layerselection 0x00000000_00000000_55555555_5755f5ff)
@@
 			)
 		)
+	)
+	(footprint "MyFootPrints:Breadboard"
+		(layer "F.Cu")
+		(at 225 166)
+		(property "Reference" "U1"
+			(at -0.05 -1.7 0)
+			(unlocked yes)
+			(layer "F.SilkS")
+			(effects
+				(font
+					(size 1 1)
+					(thickness 0.1)
+				)
+			)
+		)
+		(property "Value" "Bread Board"
+			(at -0.05 -0.2 0)
+			(unlocked yes)
+			(layer "F.Fab")
+			(effects
+				(font
+					(size 1 1)
+					(thickness 0.15)
+				)
+			)
+		)
+		(property "Datasheet" ""
+			(at 0 0 0)
+			(unlocked yes)
+			(layer "F.Fab")
+			(hide yes)
+			(effects
+				(font
+					(size 1 1)
+					(thickness 0.15)
+				)
+			)
+		)
+		(property "Description" ""
+			(at 0 0 0)
+			(unlocked yes)
+			(layer "F.Fab")
+			(hide yes)
+			(effects
+				(font
+					(size 1 1)
+					(thickness 0.15)
+				)
+			)
+		)
+		(sheetname "/")
+		(sheetfile "ProtoGuitarPedalBoard.kicad_sch")
+		(units
+			(unit
+				(name "A")
+				(pins)
+			)
+		)
+		(attr through_hole)
+		(duplicate_pad_numbers_are_jumpers no)
+		(fp_rect
+			(start -82.45 -27.5)
+			(end 82.55 27.5)
+			(stroke
+				(width 0.05)
+				(type default)
+			)
+			(fill no)
+			(layer "F.CrtYd")
+		)
+		(fp_text user "${REFERENCE}"
+			(at -0.05 1.3 0)
+			(unlocked yes)
+			(layer "F.Fab")
+			(effects
+				(font
+					(size 1 1)
+					(thickness 0.15)
+				)
+			)
+		)
+		(embedded_fonts no)
+		(model "${KIPRJMOD}/libs/models_3d/Breadboard.STEP"
+			(offset
+				(xyz 0 0 5)
+			)
+			(scale
+				(xyz 1 1 1)
+			)
+			(rotate
+				(xyz -90 -0 -0)
+			)
+		)

Commit message: Big update
Changed lines of the file:
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@@
 			(crossoutdnponfab yes)
 			(subtractmaskfromsilk no)
-			(outputformat 1)
+			(outputformat 5)
 			(mirror no)
-			(drillshape 1)
+			(drillshape 0)
 			(scaleselection 1)
-			(outputdirectory "")
+			(outputdirectory "Images/")
 		)
 	)
@@
 		)
 	)
+	(dimension
+		(type orthogonal)
+		(layer "Eco2.User")
+		(pts
+			(xy 112.5 101) (xy 337.5 101)
+		)
+		(height -4.96)
+		(orientation 0)
+		(format
+			(prefix "")
+			(suffix "")
+			(units 3)
+			(units_format 0)
+			(precision 4)
+			(suppress_zeroes yes)
+		)
+		(style
+			(thickness 0.1)
+			(arrow_length 1.27)
+			(text_position_mode 0)
+			(arrow_direction outward)
+			(extension_height 0.58642)
+			(extension_offset 0.5)
+			(keep_text_aligned yes)
+		)
+		(gr_text "225"
+			(at 225 94.89 0)
+			(layer "Eco2.User")
+			(effects
+				(font
+					(size 1 1)
+					(thickness 0.15)
+				)
+			)
+		)
+	)
+	(dimension
+		(type orthogonal)
+		(layer "Eco2.User")
+		(pts
+			(xy 337.5 101) (xy 337.5 198)
+		)
+		(height 5.49)
+		(orientation 1)
+		(format
+			(prefix "")
+			(suffix "")
+			(units 3)
+			(units_format 0)
+			(precision 4)
+			(suppress_zeroes yes)
+		)
+		(style
+			(thickness 0.1)
+			(arrow_length 1.27)
+			(text_position_mode 0)
+			(arrow_direction outward)
+			(extension_height 0.58642)
+			(extension_offset 0.5)
+			(keep_text_aligned yes)
+		)
+		(gr_text "97"
+			(at 341.84 149.5 90)
+			(layer "Eco2.User")
+			(effects
+				(font
+					(size 1 1)
+					(thickness 0.15)
+				)
+			)
+		)
+	)
 	(segment
 		(start 314 183.54)
@@
 		(polygon
 			(pts
-				(xy 100.02 99.98) (xy 350 99.98) (xy 350 199.97) (xy 100.11 199.97) (xy 100.03 199.89) (xy 100.03 99.99)
+				(xy 112.5 101) (xy 337.5 101) (xy 337.5 198) (xy 112.5 198)
 			)
 		)
