File: ProtoGuitarPedalBoard.kicad_pcb (KiCad board)
At the start: 2 copper layers, 225 x 97 mm, 25 parts, among them J1 DC_INPUT, J2 FX_IN, J3 FX_OUT, U1 Bread Board

Commit message: Update
Parts:
- moved Jack_IN1 102.6 mm to (252.9, 128.0)
- moved S1_Push_Button1 48.6 mm to (159.0, 111.7)
- moved J1 40.8 mm to (148.1, 114.1)
- moved D1_Green_LED1 38.0 mm to (169.9, 115.5)
- moved SW_3PDT_ToggleBtn1 32.3 mm to (225.0, 114.8), turned to 90 degrees
- moved D2_Red_LED1 30.9 mm to (210.1, 115.5), turned to 180 degrees
- moved R2 28.8 mm to (203.8, 110.8), turned to 0 degrees
- moved R1 23.9 mm to (166.1, 110.8)
- moved Jack_OUT1 9.39 mm to (275.9, 128.0)
- moved H1 6.46 mm to (119.7, 110.7)
- moved H2 6.24 mm to (330.6, 110.7)
- moved J_DC_Power1 4.96 mm to (151.8, 134.3)
- moved H3 2.99 mm to (119.8, 194.0)
- moved H4 2.66 mm to (330.6, 194.0)
- moved J_POT2 2.23 mm to (138.1, 183.5)
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Routing:
- net /Signal_IN: track 120.3 -> 29.8 mm
- net /DC_OUT: track 83.7 -> 22.5 mm
- net /Signal_Effect_OUT: track 73.4 -> 125.7 mm
- net /Signal_Effect_IN: track 137.5 -> 100.3 mm
- net /Signal_OUT: track 31.5 -> 53.3 mm
- net /OUT_2_LED_PWR: track 28.4 -> 7.94 mm
- net +9V: track 55.7 -> 67.1 mm
- net /LED_RED: track 20.3 -> 10.4 mm
- net Net-(D1_Green_LED1-A): track 14.8 -> 6.27 mm
- net /POT2_3: track 7.23 -> 9.45 mm
- net /POT2_2: track 7.23 -> 9.45 mm
- net /POT2_1: track 7.23 -> 9.45 mm
- net /POT1_3: track 7.33 -> 9.55 mm
- net /POT1_1: track 7.33 -> 9.55 mm
- net /POT1_2: track 7.33 -> 9.55 mm
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Other:
- board size 225 x 97 mm -> 220 x 91.3 mm
- board text added: "(DC POWER LED)"
- board text added: "(DC POWER)"
- board text added: "(GUITAR EFFECT LED)"
- board text added: "DC JACK"
- board text added: "Michał Głuszak"
- board text added: "Proto-Guitar Pedal Board"
- board text removed: "Green LED"
- board text removed: "Guitar Effect"
- board text removed: "ON/OFF (DC Power)"
- board text removed: "Red LED"
